File: src/schematics/sensor/sensor.sch (EAGLE design)
At the start: 10 parts

Commit message: Sensor PCB updates
Minor changes to the sensor module PCB layout.

Andrea Zoppi
Parts:
- R1: value 66 -> 68
- renumbered U$1 to U1
Changed lines of the file:
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@@
 <layer number="93" name="Pins" color="2" fill="1" visible="no" active="yes"/>
 <layer number="94" name="Symbols" color="4" fill="1" visible="yes" active="yes"/>
-<layer number="95" name="Names" color="7" fill="1" visible="yes" active="yes"/>
-<layer number="96" name="Values" color="7" fill="1" visible="yes" active="yes"/>
+<layer number="95" name="Names" color="15" fill="1" visible="yes" active="yes"/>
+<layer number="96" name="Values" color="15" fill="1" visible="yes" active="yes"/>
 <layer number="97" name="Info" color="7" fill="1" visible="yes" active="yes"/>
 <layer number="98" name="Guide" color="6" fill="1" visible="yes" active="yes"/>
@@
 </classes>
 <parts>
-<part name="U$1" library="avago_extended" deviceset="ADNS-2080" device=""/>
+<part name="U1" library="avago_extended" deviceset="ADNS-2080" device=""/>
 <part name="JP1" library="pinhead" deviceset="PINHD-1X5" device=""/>
-<part name="R1" library="rcl" deviceset="R-US_" device="0207/7" value="66"/>
+<part name="R1" library="rcl" deviceset="R-US_" device="0207/7" value="68"/>
 <part name="GND1" library="supply1" deviceset="GND" device=""/>
 <part name="+3V1" library="supply1" deviceset="+3V3" device=""/>
@@
 </plain>
 <instances>
-<instance part="U$1" gate="G$1" x="71.12" y="58.42"/>
+<instance part="U1" gate="G$1" x="71.12" y="58.42"/>
 <instance part="JP1" gate="A" x="-10.16" y="63.5" rot="MR0"/>
 <instance part="R1" gate="G$1" x="99.06" y="78.74" rot="R90"/>
@@
 <segment>
 <pinref part="+3V1" gate="G$1" pin="+3V3"/>
-<pinref part="U$1" gate="G$1" pin="VDDIO"/>
+<pinref part="U1" gate="G$1" pin="VDDIO"/>
 <wire x1="71.12" y1="91.44" x2="71.12" y2="88.9" width="0.1524" layer="91"/>
 <pinref part="C1" gate="G$1" pin="+"/>
@@
 <wire x1="55.88" y1="88.9" x2="71.12" y2="88.9" width="0.1524" layer="91"/>
 <wire x1="55.88" y1="86.36" x2="55.88" y2="88.9" width="0.1524" layer="91"/>
-<pinref part="U$1" gate="G$1" pin="VDDA"/>
+<pinref part="U1" gate="G$1" pin="VDDA"/>
 <wire x1="66.04" y1="71.12" x2="71.12" y2="71.12" width="0.1524" layer="91"/>
 <junction x="71.12" y="88.9"/>
@@
 <net name="N$2" class="0">
 <segment>
-<pinref part="U$1" gate="G$1" pin="VDD"/>
+<pinref part="U1" gate="G$1" pin="VDD"/>
 <wire x1="76.2" y1="71.12" x2="76.2" y2="88.9" width="0.1524" layer="91"/>
 <wire x1="76.2" y1="88.9" x2="83.82" y2="88.9" width="0.1524" layer="91"/>
@@
 </segment>
 <segment>
-<pinref part="U$1" gate="G$1" pin="GND"/>
+<pinref part="U1" gate="G$1" pin="GND"/>
 <pinref part="GND1" gate="1" pin="GND"/>
 <wire x1="71.12" y1="43.18" x2="71.12" y2="40.64" width="0.1524" layer="91"/>
@@
 <pinref part="LED1" gate="G$1" pin="C"/>
 <wire x1="99.06" y1="63.5" x2="99.06" y2="60.96" width="0.1524" layer="91"/>
-<pinref part="U$1" gate="G$1" pin="XY_LED"/>
+<pinref part="U1" gate="G$1" pin="XY_LED"/>
 <wire x1="99.06" y1="60.96" x2="93.98" y2="60.96" width="0.1524" layer="91"/>
 </segment>
@@
 <net name="MOTION" class="0">
 <segment>
-<pinref part="U$1" gate="G$1" pin="MOTION"/>
+<pinref part="U1" gate="G$1" pin="MOTION"/>
 <wire x1="93.98" y1="53.34" x2="109.22" y2="53.34" width="0.1524" layer="91"/>
 <label x="96.52" y="53.34" size="1.778" layer="95"/>
@@
 <pinref part="JP1" gate="A" pin="4"/>
 <label x="0" y="60.96" size="1.778" layer="95"/>
-<pinref part="U$1" gate="G$1" pin="SDIO"/>
+<pinref part="U1" gate="G$1" pin="SDIO"/>
 <wire x1="-7.62" y1="60.96" x2="20.32" y2="60.96" width="0.1524" layer="91"/>
 <label x="38.1" y="60.96" size="1.778" layer="95"/>
@@
 <pinref part="JP1" gate="A" pin="5"/>
 <label x="0" y="58.42" size="1.778" layer="95"/>
-<pinref part="U$1" gate="G$1" pin="SCLK"/>
+<pinref part="U1" gate="G$1" pin="SCLK"/>
 <wire x1="48.26" y1="58.42" x2="27.94" y2="58.42" width="0.1524" layer="91"/>
 <label x="38.1" y="58.42" size="1.778" layer="95"/>

Commit message: Minor PCB fixes
Changed resistor values so that performance is improved, and the PIC
inputs can read correct pull-up values.

Andrea Zoppi
Parts:
- R2, R3, R4: value 1M -> 100k; device rcl:R-US_0207/7 -> rcl:R-US_0204/5
Changed lines of the file:
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@@
 <part name="+3V3" library="supply1" deviceset="+3V3" device=""/>
 <part name="GND4" library="supply1" deviceset="GND" device=""/>
-<part name="R2" library="rcl" deviceset="R-US_" device="0207/7" value="1M"/>
-<part name="R3" library="rcl" deviceset="R-US_" device="0207/7" value="1M"/>
-<part name="R4" library="rcl" deviceset="R-US_" device="0207/7" value="1M"/>
+<part name="R2" library="rcl" deviceset="R-US_" device="0204/5" value="100k"/>
+<part name="R3" library="rcl" deviceset="R-US_" device="0204/5" value="100k"/>
+<part name="R4" library="rcl" deviceset="R-US_" device="0204/5" value="100k"/>
 </parts>
 <sheets>

Commit message: Fixed PCB libraries
Some components in the extended Microxhip library had wrong dual-in-line
package drawings.

The libraries were renamed as "local" instead of "extended".

Minor fixes in both schematics and PCBs.

Andrea Zoppi
Parts:
- U1: device avago_extended:ADNS-2080 -> avago_local:ADNS-2080
Changed lines of the file:
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@@
 </classes>
 <parts>
-<part name="U1" library="avago_extended" deviceset="ADNS-2080" device=""/>
 <part name="JP1" library="pinhead" deviceset="PINHD-1X5" device=""/>
 <part name="R1" library="rcl" deviceset="R-US_" device="0207/7" value="68"/>
@@
 <part name="R3" library="rcl" deviceset="R-US_" device="0204/5" value="100k"/>
 <part name="R4" library="rcl" deviceset="R-US_" device="0204/5" value="100k"/>
+<part name="U1" library="avago_local" deviceset="ADNS-2080" device=""/>
 </parts>
 <sheets>
@@
 </plain>
 <instances>
-<instance part="U1" gate="G$1" x="71.12" y="58.42"/>
 <instance part="JP1" gate="A" x="-10.16" y="63.5" rot="MR0"/>
 <instance part="R1" gate="G$1" x="99.06" y="78.74" rot="R90"/>
@@
 <instance part="R3" gate="G$1" x="20.32" y="71.12" rot="R90"/>
 <instance part="R4" gate="G$1" x="12.7" y="71.12" rot="R90"/>
+<instance part="U1" gate="G$1" x="71.12" y="58.42"/>
 </instances>
 <busses>
@@
 <segment>
 <pinref part="+3V1" gate="G$1" pin="+3V3"/>
-<pinref part="U1" gate="G$1" pin="VDDIO"/>
 <wire x1="71.12" y1="91.44" x2="71.12" y2="88.9" width="0.1524" layer="91"/>
 <pinref part="C1" gate="G$1" pin="+"/>
@@
 <wire x1="55.88" y1="88.9" x2="71.12" y2="88.9" width="0.1524" layer="91"/>
 <wire x1="55.88" y1="86.36" x2="55.88" y2="88.9" width="0.1524" layer="91"/>
-<pinref part="U1" gate="G$1" pin="VDDA"/>
 <wire x1="66.04" y1="71.12" x2="71.12" y2="71.12" width="0.1524" layer="91"/>
 <junction x="71.12" y="88.9"/>
 <junction x="55.88" y="88.9"/>
+<pinref part="U1" gate="G$1" pin="VDDIO"/>
 <junction x="71.12" y="71.12"/>
+<pinref part="U1" gate="G$1" pin="VDDA"/>
 </segment>
 <segment>
@@
 <net name="N$2" class="0">
 <segment>
-<pinref part="U1" gate="G$1" pin="VDD"/>
 <wire x1="76.2" y1="71.12" x2="76.2" y2="88.9" width="0.1524" layer="91"/>
 <wire x1="76.2" y1="88.9" x2="83.82" y2="88.9" width="0.1524" layer="91"/>
 <pinref part="C2" gate="G$1" pin="+"/>
 <wire x1="83.82" y1="88.9" x2="83.82" y2="86.36" width="0.1524" layer="91"/>
+<pinref part="U1" gate="G$1" pin="VDD"/>
 </segment>
 </net>
@@
 </segment>
 <segment>
-<pinref part="U1" gate="G$1" pin="GND"/>
 <pinref part="GND1" gate="1" pin="GND"/>
 <wire x1="71.12" y1="43.18" x2="71.12" y2="40.64" width="0.1524" layer="91"/>
+<pinref part="U1" gate="G$1" pin="GND"/>
 </segment>
 <segment>
@@
 <pinref part="LED1" gate="G$1" pin="C"/>
 <wire x1="99.06" y1="63.5" x2="99.06" y2="60.96" width="0.1524" layer="91"/>
+<wire x1="99.06" y1="60.96" x2="93.98" y2="60.96" width="0.1524" layer="91"/>
 <pinref part="U1" gate="G$1" pin="XY_LED"/>
-<wire x1="99.06" y1="60.96" x2="93.98" y2="60.96" width="0.1524" layer="91"/>
 </segment>
 </net>
 <net name="MOTION" class="0">
 <segment>
-<pinref part="U1" gate="G$1" pin="MOTION"/>
 <wire x1="93.98" y1="53.34" x2="109.22" y2="53.34" width="0.1524" layer="91"/>
 <label x="96.52" y="53.34" size="1.778" layer="95"/>
@@
 <wire x1="12.7" y1="66.04" x2="12.7" y2="63.5" width="0.1524" layer="91"/>
 <junction x="12.7" y="63.5"/>
+<pinref part="U1" gate="G$1" pin="MOTION"/>
 </segment>
 </net>
@@
 <pinref part="JP1" gate="A" pin="4"/>
 <label x="0" y="60.96" size="1.778" layer="95"/>
-<pinref part="U1" gate="G$1" pin="SDIO"/>
 <wire x1="-7.62" y1="60.96" x2="20.32" y2="60.96" width="0.1524" layer="91"/>
 <label x="38.1" y="60.96" size="1.778" layer="95"/>
@@
 <wire x1="20.32" y1="66.04" x2="20.32" y2="60.96" width="0.1524" layer="91"/>
 <junction x="20.32" y="60.96"/>
+<pinref part="U1" gate="G$1" pin="SDIO"/>
 </segment>
 </net>
@@
 <pinref part="JP1" gate="A" pin="5"/>
 <label x="0" y="58.42" size="1.778" layer="95"/>
-<pinref part="U1" gate="G$1" pin="SCLK"/>
 <wire x1="48.26" y1="58.42" x2="27.94" y2="58.42" width="0.1524" layer="91"/>
 <label x="38.1" y="58.42" size="1.778" layer="95"/>
@@
 <wire x1="27.94" y1="66.04" x2="27.94" y2="58.42" width="0.1524" layer="91"/>
 <junction x="27.94" y="58.42"/>
+<pinref part="U1" gate="G$1" pin="SCLK"/>
 </segment>
 </net>
