File: src/schematics/board/board.sch (EAGLE design)
At the start: 26 parts, among them P1 PN61729-S, Q1 12MHz, U1 MCP17003302E/TO, U2 PIC18LF14K50-E-P

Commit message: Incremental encoder and MOTION pins updated
Pins for incremental encoder signals (ENC_A and ENC_B), and the MOTION
signal have ben re-routed to the correct PIC pins, according to the
changes made in the latest commits.

Andrea Zoppi
Connections:
- net ENC_A: now also U2A.RC1/AN5/C12IN1-/INT1/VREFRC2/; no longer U2A.RC0/AN4/C12IN+/INT0/VREF+
- net ENC_B: now also U2A.RC2/AN6/P1D/C12IN2-/CVREF/INT2; no longer U2A.RC1/AN5/C12IN1-/INT1/VREFRC2/
- net MOTION: now also U2A.RC0/AN4/C12IN+/INT0/VREF+; no longer U2A.RC2/AN6/P1D/C12IN2-/CVREF/INT2
Other:
- moved on the sheet: R2, R3
Changed lines of the file:
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@@
 <attribute name="VALUE" x="148.59" y="58.674" size="1.778" layer="96"/>
 </instance>
-<instance part="R2" gate="G$1" x="142.24" y="25.4" rot="R90"/>
-<instance part="R3" gate="G$1" x="149.86" y="25.4" rot="R90"/>
+<instance part="R2" gate="G$1" x="144.78" y="25.4" rot="R90"/>
+<instance part="R3" gate="G$1" x="152.4" y="25.4" rot="R90"/>
 <instance part="+3V4" gate="G$1" x="170.18" y="40.64"/>
 <instance part="GND5" gate="1" x="170.18" y="20.32"/>
@@
 <wire x1="170.18" y1="33.02" x2="177.8" y2="33.02" width="0.1524" layer="91"/>
 <pinref part="R3" gate="G$1" pin="2"/>
-<wire x1="170.18" y1="33.02" x2="149.86" y2="33.02" width="0.1524" layer="91"/>
-<wire x1="149.86" y1="33.02" x2="149.86" y2="30.48" width="0.1524" layer="91"/>
+<wire x1="170.18" y1="33.02" x2="152.4" y2="33.02" width="0.1524" layer="91"/>
+<wire x1="152.4" y1="33.02" x2="152.4" y2="30.48" width="0.1524" layer="91"/>
 <pinref part="R2" gate="G$1" pin="2"/>
-<wire x1="149.86" y1="33.02" x2="142.24" y2="33.02" width="0.1524" layer="91"/>
-<wire x1="142.24" y1="33.02" x2="142.24" y2="30.48" width="0.1524" layer="91"/>
-<junction x="149.86" y="33.02"/>
+<wire x1="152.4" y1="33.02" x2="144.78" y2="33.02" width="0.1524" layer="91"/>
+<wire x1="144.78" y1="33.02" x2="144.78" y2="30.48" width="0.1524" layer="91"/>
+<junction x="152.4" y="33.02"/>
 <junction x="170.18" y="33.02"/>
 </segment>
@@
 <net name="ENC_A" class="0">
 <segment>
-<pinref part="U2" gate="A" pin="RC0/AN4/C12IN+/INT0/VREF+"/>
-<label x="127" y="17.78" size="1.778" layer="95"/>
 <pinref part="P3" gate="A" pin="2"/>
 <wire x1="177.8" y1="30.48" x2="157.48" y2="30.48" width="0.1524" layer="91"/>
-<wire x1="157.48" y1="30.48" x2="157.48" y2="17.78" width="0.1524" layer="91"/>
-<wire x1="157.48" y1="17.78" x2="142.24" y2="17.78" width="0.1524" layer="91"/>
+<wire x1="157.48" y1="30.48" x2="157.48" y2="15.24" width="0.1524" layer="91"/>
+<wire x1="157.48" y1="15.24" x2="144.78" y2="15.24" width="0.1524" layer="91"/>
 <pinref part="R2" gate="G$1" pin="1"/>
-<wire x1="142.24" y1="17.78" x2="124.46" y2="17.78" width="0.1524" layer="91"/>
-<wire x1="142.24" y1="20.32" x2="142.24" y2="17.78" width="0.1524" layer="91"/>
-<junction x="142.24" y="17.78"/>
+<wire x1="144.78" y1="20.32" x2="144.78" y2="15.24" width="0.1524" layer="91"/>
 <label x="162.56" y="30.48" size="1.778" layer="95"/>
+<pinref part="U2" gate="A" pin="RC1/AN5/C12IN1-/INT1/VREFRC2/"/>
+<wire x1="124.46" y1="15.24" x2="144.78" y2="15.24" width="0.1524" layer="91"/>
+<junction x="144.78" y="15.24"/>
+<label x="127" y="15.24" size="1.778" layer="95"/>
 </segment>
 </net>
 <net name="ENC_B" class="0">
 <segment>
-<pinref part="U2" gate="A" pin="RC1/AN5/C12IN1-/INT1/VREFRC2/"/>
-<label x="127" y="15.24" size="1.778" layer="95"/>
-<wire x1="124.46" y1="15.24" x2="149.86" y2="15.24" width="0.1524" layer="91"/>
-<wire x1="149.86" y1="15.24" x2="160.02" y2="15.24" width="0.1524" layer="91"/>
-<wire x1="160.02" y1="15.24" x2="160.02" y2="27.94" width="0.1524" layer="91"/>
+<wire x1="152.4" y1="12.7" x2="160.02" y2="12.7" width="0.1524" layer="91"/>
+<wire x1="160.02" y1="12.7" x2="160.02" y2="27.94" width="0.1524" layer="91"/>
 <pinref part="P3" gate="A" pin="3"/>
 <wire x1="160.02" y1="27.94" x2="177.8" y2="27.94" width="0.1524" layer="91"/>
 <pinref part="R3" gate="G$1" pin="1"/>
-<wire x1="149.86" y1="20.32" x2="149.86" y2="15.24" width="0.1524" layer="91"/>
-<junction x="149.86" y="15.24"/>
+<wire x1="152.4" y1="20.32" x2="152.4" y2="12.7" width="0.1524" layer="91"/>
 <label x="162.56" y="27.94" size="1.778" layer="95"/>
+<pinref part="U2" gate="A" pin="RC2/AN6/P1D/C12IN2-/CVREF/INT2"/>
+<wire x1="152.4" y1="12.7" x2="124.46" y2="12.7" width="0.1524" layer="91"/>
+<junction x="152.4" y="12.7"/>
+<label x="127" y="12.7" size="1.778" layer="95"/>
 </segment>
 </net>
 <net name="MOTION" class="0">
-<segment>
-<pinref part="U2" gate="A" pin="RC2/AN6/P1D/C12IN2-/CVREF/INT2"/>
-<wire x1="137.16" y1="12.7" x2="124.46" y2="12.7" width="0.1524" layer="91"/>
-<label x="127" y="12.7" size="1.778" layer="95"/>
-</segment>
 <segment>
 <pinref part="P5" gate="A" pin="3"/>
 <wire x1="177.8" y1="60.96" x2="160.02" y2="60.96" width="0.1524" layer="91"/>
 <label x="162.56" y="60.96" size="1.778" layer="95"/>
-</segment>
-</net>
+<wire x1="160.02" y1="60.96" x2="160.02" y2="45.72" width="0.1524" layer="91"/>
+<pinref part="U2" gate="A" pin="RC0/AN4/C12IN+/INT0/VREF+"/>
+<wire x1="137.16" y1="17.78" x2="124.46" y2="17.78" width="0.1524" layer="91"/>
+<label x="127" y="17.78" size="1.778" layer="95"/>
+<wire x1="160.02" y1="45.72" x2="137.16" y2="45.72" width="0.1524" layer="91"/>
+<wire x1="137.16" y1="45.72" x2="137.16" y2="17.78" width="0.1524" layer="91"/>
+</segment>
+</net>

Commit message: Fixed PCB libraries
Some components in the extended Microxhip library had wrong dual-in-line
package drawings.

The libraries were renamed as "local" instead of "extended".

Minor fixes in both schematics and PCBs.

Andrea Zoppi
Parts:
- U1: value MCP17003302E/TO -> PIC18F14K50-E-P; device microchip_extended:MCP17003302E/TO -> microchip_local:PIC18F14K50-E-P
- U2: value PIC18LF14K50-E-P -> MCP17003302E/TO; device microchip_extended:PIC18F14K50-E-P -> microchip_local:MCP17003302E/TO
Connections:
- removed net ENC_A: P3.2, R2.1, U2A.RC1/AN5/C12IN1-/INT1/VREFRC2/
- removed net ENC_B: P3.3, R3.1, U2A.RC2/AN6/P1D/C12IN2-/CVREF/INT2
- new net QA: P3.3, R2.1, U1A.RC1/AN5/C12IN1-/INT1/VREFRC2/
- new net QB: P3.4, R3.1, U1A.RC2/AN6/P1D/C12IN2-/CVREF/INT2
- net +3V3: now also P3.2, U1A.VUSB, U1P.VDD, U2.OUT; no longer P3.1, U1.OUT, U2A.VUSB, U2P.VDD
- net +5V: now also U2.IN; no longer U1.IN
- net AUXIN: now also U1A.RC6/AN8/*SS/T13CKI/T1OSCI; no longer U2A.RC6/AN8/*SS/T13CKI/T1OSCI
- net D+: now also U1A.RA0/D+/PGD; no longer U2A.RA0/D+/PGD
- net D-: now also U1A.RA1/D-/PGC; no longer U2A.RA1/D-/PGC
- net GND: now also P3.1, U1P.VSS, U2.GND; no longer P3.4, U1.GND, U2P.VSS
- net GREEN: now also U1A.RC3/AN7/P1C/C12IN3-/PGM; no longer U2A.RC3/AN7/P1C/C12IN3-/PGM
- net MOSI: now also U1A.RC7/AN9/SDO/T1OSCO; no longer U2A.RC7/AN9/SDO/T1OSCO
- net MOTION: now also U1A.RC0/AN4/C12IN+/INT0/VREF+; no longer U2A.RC0/AN4/C12IN+/INT0/VREF+
- net N$2: now also U1A.RA4/AN3/OSC2/CLKOUT; no longer U2A.RA4/AN3/OSC2/CLKOUT
- net N$3: now also U1A.RA5/OSC1/CLKIN; no longer U2A.RA5/OSC1/CLKIN
- net RED: now also U1A.RC5/CCP1/P1A/T0CKI; no longer U2A.RC5/CCP1/P1A/T0CKI
- net RST: now also U1A.RA3/*MCLR/VPP; no longer U2A.RA3/*MCLR/VPP
- net RX: now also U1A.RB5/AN11/RX/DT; no longer U2A.RB5/AN11/RX/DT
- net SCLK: now also U1A.RB6/SCK/SCL; no longer U2A.RB6/SCK/SCL
- net SDIO: now also U1A.RB4/AN10/SDI/SDA; no longer U2A.RB4/AN10/SDI/SDA
- net TX: now also U1A.RB7/TX/CK; no longer U2A.RB7/TX/CK
- net YELLOW: now also U1A.RC4/P1B/C12OUT/SRQ; no longer U2A.RC4/P1B/C12OUT/SRQ
Other:
- moved on the sheet: P3, R2, R3
